File: Placa_cobre/Placa_cobre.kicad_sch (KiCad schematic)
At the start: 3 parts

Commit message: codigo funcional, mandando e recebendo sinal, recpetor e transmissor
Parts:
- removed U1: ~, symbol RF_transmissor_receptor:RF_RECEPTOR
- removed U2: ~, symbol RF_transmissor_receptor:rf_transmissor
- added J1: Conn_01x03_Socket, Connector_PinSocket_2.54mm:PinSocket_1x03_P2.54mm_Vertical, symbol Connector:Conn_01x03_Socket
- added J2: Conn_01x04_Socket, Connector_PinSocket_2.54mm:PinSocket_1x04_P2.54mm_Vertical, symbol Connector:Conn_01x04_Socket
- added SW1, SW2: Push_Button, Button_Switch_THT:SW_PUSH_6mm, symbol PCM_SL_Devices:Push_Button
Connections:
- net 3.3V: now reaches A1.1 (3.3V)
- net RX_RECEPTOR: now reaches A1.12 (RX0/GPIO3)
- net RX_RECEPTOR: now also J2.2 (Pin_2)
- net TX_TRANSMISSOR: now reaches A1.13 (TX0/GPIO1)
- net TX_TRANSMISSOR: now also J1.1 (Pin_1)
- net GND: now reaches A1.2 (GND)
- net GND: now also A1.29 (GND), J1.3 (Pin_3), J2.4 (Pin_4), SW1.2, SW2.2
- net VIN: now reaches A1.30 (VIN)
- net VIN: now also J1.2 (Pin_2), J2.1 (Pin_1)
- new net BUTTON_1: SW1.1
- new net BUTTON_2: SW2.1
- new net RX_RECEPTOR_1: J2.3 (Pin_3)

Commit message: tranasmissor mandado certo para o receptor
Connections:
- net BUTTON_1: now also A1.17 (ADC1_CH0/VP)
- net BUTTON_2: now also A1.15 (D23)
Changed lines of the file:
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@@
 	(global_label "BUTTON_1"
 		(shape input)
-		(at 44.45 39.37 180)
+		(at 105.41 99.06 0)
 		(fields_autoplaced yes)
 		(effects
@@
 				(size 1.27 1.27)
 			)
-			(justify right)
+			(justify left)
 		)
 		(property "Intersheetrefs" "${INTERSHEET_REFS}"
-			(at 32.091 39.37 0)
+			(at 117.769 99.06 0)
 			(effects
 				(font
 					(size 1.27 1.27)
 				)
-				(justify right)
+				(justify left)
 				(hide yes)
 			)
@@
 				)
 				(justify left)
+				(hide yes)
+			)
+		)
+	)
+	(global_label "BUTTON_2"
+		(shape input)
+		(at 60.96 101.6 180)
+		(fields_autoplaced yes)
+		(effects
+			(font
+				(size 1.27 1.27)
+			)
+			(justify right)
+		)
+		(property "Intersheetrefs" "${INTERSHEET_REFS}"
+			(at 48.601 101.6 0)
+			(effects
+				(font
+					(size 1.27 1.27)
+				)
+				(justify right)
 				(hide yes)
 			)
@@
 			(effects
 				(font
+					(size 1.27 1.27)
+				)
+				(justify right)
+				(hide yes)
+			)
+		)
+	)
+	(global_label "BUTTON_1"
+		(shape input)
+		(at 44.45 39.37 180)
+		(fields_autoplaced yes)
+		(effects
+			(font
+				(size 1.27 1.27)
+			)
+			(justify right)
+		)
+		(property "Intersheetrefs" "${INTERSHEET_REFS}"
+			(at 32.091 39.37 0)
+			(effects
+				(font
